File: hardware/ui/sendspin-speaker-ui.kicad_sch (KiCad schematic)
At the start: 0 parts

Commit message: hardware: split into main, front panel and USB-C boards
Three KiCad projects (main/, ui/, usb/) sharing hardware/lib/. JST
connector plan for the front panel, USB-C board (or USB-C on the main
board), LiPo, speakers and status LED; 0805 for SMD passives and LEDs
wherever possible.

Co-Authored-By: Claude Opus 5.5 <noreply@anthropic.com>
Other:
- title: ESP32 Sendspin Speaker -> ESP32 Sendspin Speaker — front panel (display + buttons)
Changed lines of the file:
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@@
 	(generator "eeschema")
 	(generator_version "9.0")
-	(paper "A3")
+	(paper "A4")
 	(title_block
-		(title "ESP32 Sendspin Speaker")
+		(title "ESP32 Sendspin Speaker — front panel (display + buttons)")
 		(date "2026-10-30")
 		(rev "A")
