File: hardware/usb/sendspin-speaker-usb.kicad_sch (KiCad schematic)
At the start: 0 parts

Commit message: hardware: front panel and USB-C board schematics; docs
All three projects pass ERC with 0 violations and every part has its
footprint. Open checks (PJ-320D pinout, NS4150B values) in the README.

Co-Authored-By: Claude Opus 5.5 <noreply@anthropic.com>
Parts:
- added J701: J_USB, Connector_JST:JST_XH_B4B-XH-A_1x04_P2.50mm_Vertical, symbol Connector_Generic:Conn_01x04
- added R701, R702: 5.1k, Resistor_SMD:R_0805_2012Metric, symbol Device:R
- added U701: USBLC6-2SC6, Package_TO_SOT_SMD:SOT-23-6, symbol Power_Protection:USBLC6-2SC6
- added USB701: USB-C, Connector_USB:USB_C_Receptacle_HRO_TYPE-C-31-M-12, symbol Connector:USB_C_Receptacle_USB2.0_16P
Connections:
- new net CC1: R701.1, USB701.A5 (CC1)
- new net CC2: R702.1, USB701.B5 (CC2)
- new net GND: J701.4 (Pin_4), R701.2, R702.2, U701.2 (GND), USB701.A1 (GND), USB701.A12 (GND), USB701.B1 (GND), USB701.B12 (GND), USB701.SH (SHIELD)
- new net USB_DN: J701.2 (Pin_2), U701.3 (I/O2), U701.4 (I/O2), USB701.A7 (D-), USB701.B7 (D-)
- new net USB_DP: J701.3 (Pin_3), U701.1 (I/O1), U701.6 (I/O1), USB701.A6 (D+), USB701.B6 (D+)
- new net VBUS: J701.1 (Pin_1), U701.5 (VBUS), USB701.A4 (VBUS), USB701.A9 (VBUS), USB701.B4 (VBUS), USB701.B9 (VBUS)
- no-connect marks 0 -> 2
Other:
- note added: "USB-C board Receptacle, 5.1k on CC1 and CC2 separately (5 V sink), USBLC6-2SC6 next to the receptacle. J701 to the main board's J_USB (XH 4: VBUS, D-, D+, GND). Cable <= 15 cm for USB full speed. Fit this board or USB301 on the main board, not both."

Commit message: hardware: bare USB-C board and front panel (schematics)
J_USB carries CC1/CC2 (XH 6); CC resistors and ESD stay on the main
board. Front panel has only buttons and headers; its LED pin comes
through R501. Boards not yet updated from the schematics.

Co-Authored-By: Claude Opus 5.5 <noreply@anthropic.com>
Parts:
- removed J701: J_USB, Connector_JST:JST_XH_B4B-XH-A_1x04_P2.50mm_Vertical, symbol Connector_Generic:Conn_01x04
- removed R701, R702: 5.1k, Resistor_SMD:R_0805_2012Metric, symbol Device:R
- removed U701: USBLC6-2SC6, Package_TO_SOT_SMD:SOT-23-6, symbol Power_Protection:USBLC6-2SC6
- added J701: J_USB, Connector_JST:JST_XH_B6B-XH-A_1x06_P2.50mm_Vertical, symbol Connector_Generic:Conn_01x06
Connections:
- net CC1: now also J701.4 (Pin_4)
- net CC2: now also J701.5 (Pin_5)
- net GND: now also J701.6 (Pin_6)
- net USB_DN: now also J701.2 (Pin_2)
- net USB_DP: now also J701.3 (Pin_3)
- net VBUS: now also J701.1 (Pin_1)
Other:
- note added: "USB-C board Bare breakout: receptacle and J701 only, no parts. The 5.1k CC resistors and the ESD sit on the main board, so any USB-C breakout or panel socket that brings out VBUS, D-, D+, CC1, CC2 and GND can replace this board (without its own 5.1k, or leave R301/R302 off). J701 to the main board's J_USB (XH 6). Cable <= 15 cm for USB full speed. Fit this board or USB301 on the main board, not b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"
- note removed: "USB-C board Receptacle, 5.1k on CC1 and CC2 separately (5 V sink), USBLC6-2SC6 next to the receptacle. J701 to the main board's J_USB (XH 4: VBUS, D-, D+, GND). Cable <= 15 cm for USB full speed. Fit this board or USB301 on the main board, not both."
