File: hardware/main/power.kicad_sch (KiCad schematic)
At the start: 30 parts, among them J201 J_BAT, J202 J_SW, J203 J_CHG, Q201 FS8205A, Q202 AO3401A, SW201 MSK12C02, U201 TP4056, U202 DW01A, U203 AP2112K-3.3

Commit message: hardware: main board routed and labelled, JLC files
- Freerouting (jar, portable Java 25) via scripts/route.py; net classes
  Power 0.8 mm / Supply 0.4 mm so tracks fit the fine-pitch pins.
- Silkscreen pin names and function labels (silk_main.py), references on
  the fab layer, SMD GND pads solid to the pour; board 100 x 58 mm.
- LCSC numbers on all SMD parts (checked on lcsc.com); jlc.py writes the
  Gerber ZIP, BOM and CPL in JLC's formats.

Co-Authored-By: Claude Opus 5.5 <noreply@anthropic.com>
Parts:
- C201, C202, C204, C205, C206: LCSC (none) -> C15850
- C203, C207: LCSC (none) -> C49678
- D201: LCSC (none) -> C84256
- D202: LCSC (none) -> C2297
- D203, D204: LCSC (none) -> C2992467
- D205: LCSC (none) -> C8678
- Q202: LCSC (none) -> C15127
- R201: LCSC (none) -> C17526
- R202, R203, R205: LCSC (none) -> C17513
- R204: LCSC (none) -> C17408
- R206: LCSC (none) -> C149504
- R207, R208: LCSC (none) -> C17709
- U201: LCSC (none) -> C16581
- U202: LCSC (none) -> C351410
- U203: LCSC (none) -> C51118
Changed lines of the file:
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@@
 			)
 		)
+		(property "LCSC" "C84256"
+			(at 0 0 0)
+			(hide yes)
+			(effects
+				(font
+					(size 1.27 1.27)
+				)
+			)
+		)
 		(property "Description" ""
 			(at 40.64 125.73 0)
@@
 			)
 		)
+		(property "LCSC" "C15850"
+			(at 0 0 0)
+			(hide yes)
+			(effects
+				(font
+					(size 1.27 1.27)
+				)
+			)
+		)
 		(property "Description" ""
 			(at 236.22 160.02 0)
@@
 			)
 		)
+		(property "LCSC" "C351410"
+			(at 0 0 0)
+			(hide yes)
+			(effects
+				(font
+					(size 1.27 1.27)
+				)
+			)
+		)
 		(property "Description" ""
 			(at 220.98 63.5 0)
@@
 			)
 		)
+		(property "LCSC" "C15850"
+			(at 0 0 0)
+			(hide yes)
+			(effects
+				(font
+					(size 1.27 1.27)
+				)
+			)
+		)
 		(property "Description" ""
 			(at 322.58 99.06 0)
@@
 			)
 		)
+		(property "LCSC" "C2992467"
+			(at 0 0 0)
+			(hide yes)
+			(effects
+				(font
+					(size 1.27 1.27)
+				)
+			)
+		)
 		(property "Description" ""
 			(at 116.84 125.73 0)
@@
 			)
 		)
+		(property "LCSC" "C17526"
+			(at 0 0 0)
+			(hide yes)
+			(effects
+				(font
+					(size 1.27 1.27)
+				)
+			)
+		)
 		(property "Description" ""
 			(at 110.49 80.01 0)
@@
 			)
 		)
+		(property "LCSC" "C17513"
+			(at 0 0 0)
+			(hide yes)
+			(effects
+				(font
+					(size 1.27 1.27)
+				)
+			)
+		)
 		(property "Description" ""
 			(at 254 76.2 0)
@@
 			)
 		)
+		(property "LCSC" "C15850"
+			(at 0 0 0)
+			(hide yes)
+			(effects
+				(font
+					(size 1.27 1.27)
+				)
+			)
+		)
 		(property "Description" ""
 			(at 125.73 80.01 0)
@@
 			)
 		)
+		(property "LCSC" "C2297"
+			(at 0 0 0)
+			(hide yes)
+			(effects
+				(font
+					(size 1.27 1.27)
+				)
+			)
+		)
 		(property "Description" ""
 			(at 40.64 151.13 0)
@@
 			)
 		)
+		(property "LCSC" "C49678"
+			(at 0 0 0)
+			(hide yes)
+			(effects
+				(font
+					(size 1.27 1.27)
+				)
+			)
+		)
 		(property "Description" ""
 			(at 271.78 50.8 0)
@@
 			)
 		)
+		(property "LCSC" "C2992467"
+			(at 0 0 0)
+			(hide yes)
+			(effects
+				(font
+					(size 1.27 1.27)
+				)
+			)
+		)
 		(property "Description" ""
 			(at 116.84 151.13 0)
@@
 			)
 		)
+		(property "LCSC" "C149504"
+			(at 0 0 0)
+			(hide yes)
+			(effects
+				(font
+					(size 1.27 1.27)
+				)
+			)
+		)
 		(property "Description" ""
 			(at 218.44 160.02 0)
@@
 			)
 		)
+		(property "LCSC" "C17513"
+			(at 0 0 0)
+			(hide yes)
+			(effects
+				(font
+					(size 1.27 1.27)
+				)
+			)
+		)
 		(property "Description" ""
 			(at 76.2 154.94 0)
@@
 			)
 		)
+		(property "LCSC" "C17513"
+			(at 0 0 0)
+			(hide yes)
+			(effects
+				(font
+					(size 1.27 1.27)
+				)
+			)
+		)
 		(property "Description" ""
 			(at 76.2 129.54 0)
@@
 			)
 		)
+		(property "LCSC" "C17408"
+			(at 0 0 0)
+			(hide yes)
+			(effects
+				(font
+					(size 1.27 1.27)
+				)
+			)
+		)
 		(property "Description" ""
 			(at 254 50.8 0)
@@
 			)
 		)
+		(property "LCSC" "C15850"
+			(at 0 0 0)
+			(hide yes)
+			(effects
+				(font
+					(size 1.27 1.27)
+				)
+			)
+		)
 		(property "Description" ""
 			(at 370.84 99.06 0)
@@
 			)
 		)
+		(property "LCSC" "C17709"
+			(at 0 0 0)
+			(hide yes)
+			(effects
+				(font
+					(size 1.27 1.27)
+				)
+			)
+		)
 		(property "Description" ""
 			(at 330.2 172.72 0)
@@
 			)
 		)
+		(property "LCSC" "C15850"
+			(at 0 0 0)
+			(hide yes)
+			(effects
+				(font
+					(size 1.27 1.27)
+				)
+			)
+		)
 		(property "Description" ""
 			(at 50.8 55.88 0)
@@
 			)
 		)
+		(property "LCSC" "C8678"
+			(at 0 0 0)
+			(hide yes)
+			(effects
+				(font
+					(size 1.27 1.27)
+				)
+			)
+		)
 		(property "Description" ""
 			(at 190.5 147.32 0)
@@
 			)
 		)
+		(property "LCSC" "C49678"
+			(at 0 0 0)
+			(hide yes)
+			(effects
+				(font
+					(size 1.27 1.27)
+				)
+			)
+		)
 		(property "Description" ""
 			(at 355.6 172.72 0)
@@
 			)
 		)
+		(property "LCSC" "C51118"
+			(at 0 0 0)
+			(hide yes)
+			(effects
+				(font
+					(size 1.27 1.27)
+				)
+			)
+		)
 		(property "Description" ""
 			(at 345.44 80.01 0)
@@
 			)
 		)
+		(property "LCSC" "C16581"
+			(at 0 0 0)
+			(hide yes)
+			(effects
+				(font
+					(size 1.27 1.27)
+				)
+			)
+		)
 		(property "Description" ""
 			(at 80.01 80.01 0)
@@
 			)
 		)
+		(property "LCSC" "C15127"
+			(at 0 0 0)
+			(hide yes)
+			(effects
+				(font
+					(size 1.27 1.27)
+				)
+			)
+		)
 		(property "Description" ""
 			(at 190.5 175.26 0)
@@
 			(effects
 				(font
+					(size 1.27 1.27)
+				)
+			)
+		)
+		(property "LCSC" "C17709"
+			(at 0 0 0)
+			(hide yes)
+			(effects
+				(font
